File: front_panel.kicad_pcb (KiCad board)
At the start: 2 copper layers, 81.9 x 30 mm, 0 parts

Commit message: man, this is a pretty tight fit ...
Other:
- outline, holes or cut-outs redrawn
Changed lines of the file:
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@@
     (uvia_drill 0.1)
   )
-  (gr_text "CUTOUT\n" (at 137.5 110.5) (layer F.Mask)
+  (gr_text "CUTOUT\n" (at 137.5 111.5) (layer F.Mask)
     (effects (font (size 1 1) (thickness 0.15)))
   )
-  (gr_circle (center 137.5 110.35) (end 144 110.35) (layer Edge.Cuts) (width 0.05))
+  (gr_circle (center 137.5 111.35) (end 144 111.35) (layer Edge.Cuts) (width 0.05))
   (gr_text INPUT (at 137.5 123.8) (layer F.Mask)
     (effects (font (size 3 3) (thickness 0.6)))
@@
   (gr_poly (pts (xy 179 130.5) (xy 96 130.5) (xy 96 99.5) (xy 179 99.5)) (layer B.Cu) (width 0.1))
   (gr_poly (pts (xy 179 130.5) (xy 96 130.5) (xy 96 99.5) (xy 179 99.5)) (layer F.Cu) (width 0.1))
-  (gr_circle (center 137.5 110.35) (end 144.5 110.35) (layer F.Mask) (width 4))
+  (gr_circle (center 137.5 111.35) (end 144.5 111.35) (layer F.Mask) (width 4))
   (gr_arc (start 129.999421 114.998265) (end 99.153372 127.946947) (angle 45.5406599) (layer Edge.Cuts) (width 0.05))
   (gr_arc (start 102 127) (end 102 130) (angle 71.6) (layer Edge.Cuts) (width 0.05))
