File: mu_lna.kicad_pcb (KiCad board)
At the start: 2 copper layers, 100 x 77.8 mm, 55 parts, among them J3 Conn_01x02, J4 Conn_01x02, J5 Conn_01x01, SW1 SWW246/7, U1 ADA4523-1, U2 Opamp_Dual_Generic, U3 ADA4523-1, U4 ADA4523-1, U5 ADA4523-1

Commit message: man, this is a pretty tight fit ...
Parts:
- moved BT1 1.00 mm to (131.2, 111.8)
- moved BT2 1.00 mm to (158.7, 111.8)
- moved C12 1.00 mm to (105.8, 77.2)
Routing:
- net Net-(C12-Pad2): track 70.1 -> 61.6 mm
- net Net-(BT2-Pad2): track 87.0 -> 88.0 mm
- net Net-(C12-Pad1): track 28.4 -> 27.4 mm
